File: Hardware/project-tsc.brd (EAGLE design)
At the start: 160 x 100 mm, 105 parts, among them IC1 BQ25180YBGR, IC2 DRV2605YZFR, IC3 BMA421, IC9 RT6160AWSC, J1 TC2030-IDC_TC2030-IDC, J2 503480-2400_503480-2400, J4 KH-TYPE-C-16P, Q3 SI1308EDL-T1-GE3, U1 NRF52840_QF, U2 ESP32_C6_LIBRARY_MAX17048G+T10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

Commit message: Add system block diagram for InkTime Smartwatch in SVG format
- Created a detailed SVG block diagram illustrating the system architecture of the InkTime Smartwatch.
- Included components : MCU, E-Paper Display, IMU, Haptic Driver, USB-C, Battery, Fuel Gauge, and Power Management ICs.
- Added connection lines and labels for various interfaces (SPI, I2C, GPIO) to enhance clarity.
- Implemented a legend for easy reference to connection types and signal paths.
Parts:
- removed DMG2305UX-7: 20V/4.2A/52mΩ/1.4W, InkTime_v5:ESP32_C6_LIBRARY_4_ESP32_C6_LIBRARY_4_ESP32_C6_LIBRARY_4_ESP32_C6_LIBRARY_4_ESP32_WROVER_SPARKFUN-DISCRETESE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
- removed R4, R6: 10K, InkTime_v5:CPF0201D7K68C1_0201
- removed U$16: 3.9nH, InkTime_v5:NORDIC_NRF_2_RESC0402_L
- added L1: 3.9nH, InkTime_v5:NORDIC_NRF_2_RESC0402_L
- added Q1: 20V/4.2A/52mΩ/1.4W, InkTime_v5:ESP32_C6_LIBRARY_4_ESP32_C6_LIBRARY_4_ESP32_C6_LIBRARY_4_ESP32_C6_LIBRARY_4_ESP32_WROVER_SPARKFUN-DISCRETESE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
- added R7, R8: 10K, InkTime_v5:CPF0201D7K68C1_0201
- moved ANT1 229.2 mm to (18.5, -13.3), turned to 270 degrees
- moved C1 213.3 mm to (21.3, -3.47), turned to 180 degrees
- moved L3\ 202.1 mm to (21.8, 1.37)
- moved TP_SWDCLK 200.5 mm to (9.03, 11.3)
- moved C4 200.0 mm to (15.2, -9.52), turned to 180 degrees
- moved TP_3V3 197.6 mm to (-4.97, -9.87)
- moved C22 196.6 mm to (19.3, -9.62)
- moved L2 196.5 mm to (19.9, 1.37)
- moved TP_OP 196.5 mm to (6.63, 11.3)
- moved C3 196.2 mm to (15.4, -8.40), turned to 270 degrees
- moved R18 191.4 mm to (1.18, -8.27)
- moved TP_ON 191.3 mm to (9.25, 13.7)
- moved TP_SCL 190.8 mm to (-6.29, -7.28)
- moved C7 190.5 mm to (10.7, -8.75), turned to 180 degrees
- moved R17 190.0 mm to (-0.27, -8.44)
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Connections:
- removed net EDP_3V3: DMG2305UX-7.3
- removed net N$72: C8.2
- net 3V3: now also Q1.2, R7.1, R8.1; no longer DMG2305UX-7.2, R4.1, R6.1
- net EPD_3V3: now also Q1.3
- net GND: now also C8.2
- net N$74: now also L1.2; no longer U$16.2
- net N$75: now also L1.1; no longer U$16.1
- net P0.14: now also R8.2; no longer R4.2
- net P1.01: now also Q1.1; no longer DMG2305UX-7.1
- net P1.02: now also R7.2; no longer R6.2
Routing:
- net 3V3: track 0.00 -> 129.2 mm, vias 0 -> 7
- net SWDIO: track 0.00 -> 53.2 mm, vias 0 -> 3
- net VBUS: track 0.00 -> 51.7 mm, vias 0 -> 3
- net SCL: track 0.00 -> 49.9 mm, vias 0 -> 5
- net SCK: track 0.00 -> 47.1 mm, vias 0 -> 2
- net SDA: track 0.00 -> 44.2 mm, vias 0 -> 2
- net SWDCLK: track 0.00 -> 39.4 mm, vias 0 -> 3
- net PREVGH: track 0.00 -> 39.2 mm, vias 0 -> 2
- net P1.02: track 0.00 -> 36.4 mm, vias 0 -> 3
- net ALERT: track 0.00 -> 35.3 mm, vias 0 -> 2
- net VREG: track 0.00 -> 30.4 mm, vias 0 -> 2
- net EPD_BUSY: track 0.00 -> 26.7 mm, vias 0 -> 3
- net GND: track 0.00 -> 26.3 mm
- net D-: track 0.00 -> 25.8 mm, vias 0 -> 3
- net P0.14: track 0.00 -> 25.1 mm, vias 0 -> 2
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- added copper zone on layer 1, net GND
- added copper zone on layer 16, net GND
- added copper zone on layer 2, net GND
Other:
- board size 160 x 100 mm -> 46 x 35 mm

Commit message: Refactor code structure for improved readability and maintainability
Parts:
- EDP_C1, EDP_C2: value 10uF -> 1uF
- R1, R2: value 10K -> 0
- moved R5 2.10 mm to (7.96, -1.74)
- moved C17 0.94 mm to (17.5, 1.91)
- moved C5 0.73 mm to (16.6, 1.57)
- moved C18\ 0.69 mm to (15.6, 1.67)
- moved C6 0.30 mm to (10.2, -4.23)
- moved C20 0.23 mm to (10.8, 0.88)
Routing:
- net GND: track 26.3 -> 805.8 mm, vias 0 -> 58
- net EPD_RST: track 0.00 -> 53.8 mm, vias 0 -> 4
- net EPD_CS: track 0.00 -> 45.1 mm, vias 0 -> 2
- net MOSI: track 0.00 -> 40.8 mm, vias 0 -> 4
- net RESET: track 13.9 -> 50.1 mm, vias 0 -> 2
- net P1.01: track 2.77 -> 32.6 mm, vias 0 -> 2
- net PMIC_INT: track 0.00 -> 27.7 mm, vias 0 -> 2
- net EPD_DC: track 0.00 -> 26.2 mm, vias 0 -> 2
- net P0.13: track 3.41 -> 28.0 mm, vias 0 -> 2
- net IMU_INT2: track 0.00 -> 20.5 mm, vias 0 -> 2
- net N$3: track 8.44 -> 20.1 mm, vias 0 -> 2
- net VREG: track 30.4 -> 38.6 mm
- net VBUS: track 51.7 -> 45.7 mm
- net SCL: track 49.9 -> 55.8 mm
- net 3V3: track 129.2 -> 125.6 mm
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